File: hw/eagle/FMC_P_CAM.sch (EAGLE design)
At the start: 1 part, among them J1 FMC-LPC

Commit message: update board
Parts:
- added U1: SN74AVCH16T245_DGV_48, SN74AVCH16T245_DGV_48:SN74AVCH16T245_DGV_48
- J1: OC_NEWARK (none) -> unknown
Connections:
- removed net VADJ: J1H.VADJ@H40
- net FMC_CAM1_RSVD0: now also U1.2B7
- net FMC_CAM1_RSVD1: now also U1.2B6
- net FMC_CAM1_RSVD2: now also U1.2B5
- net FMC_CAM1_RSVD3: now also U1.2B4
- net FMC_CAM1_RSVD4: now also U1.2B3
- net FMC_CAM1_RSVD6: now also U1.2B1
- net GND: now also U1.GND, U1.GND_2, U1.GND_3, U1.GND_4, U1.GND_5, U1.GND_6, U1.GND_7, U1.GND_8
- net VDD: now also J1H.VADJ@H40, U1.VCCA, U1.VCCA_2, U1.VCCB, U1.VCCB_2
