File: hw/eagle/FMC_P_CAM.sch (EAGLE design)
At the start: 2 parts, among them J1 FMC-LPC, U1 SN74AVCH16T245_DGV_48

Commit message: update schematic
Parts:
- added C1, C2, C3, C4, C5, C6, C7: (no value), resistor:C-EUC0603
- added C10, C11, C12, C13, C14, C15, C16, C8, C9: (no value), my-rcl:C-EUC0603
- added LED1: LY_T679-D2E2-1, led:LY_T679-D2E2-1
- added R1, R2, R3: 4K7, resistor:R-EU_R0603
- added R4, R5, R6, R7, R8: (no value), resistor:R-EU_R0603
- added U$10, U$12: L-MY, my-rcl:L-MY
- added U$8: (no value), CX5032GB (CX-53F):CX5032GB27000
- added U2: SN74LVC1G14_DCK_5, SN74LVC1G14_DCK_5:SN74LVC1G14_DCK_5
- added U3: PCA9546A_DGV_16, PCA9546A_DGV_16:PCA9546A_DGV_16
- added U4: CDCE925_PW_16, CDCE925_PW_16:CDCE925_PW_16
- added U5: TPS71718_DCK_5, TPS71718_DCK_5:TPS71718_DCK_5
Connections:
- net +12V renamed 12P0V
- removed net +3V3: J1C.3P3V@C39, J1D.3P3V@D36, J1D.3P3V@D38, J1D.3P3V@D40
- removed net VDD: J1G.VADJ@G39, J1H.VADJ@H40, U1.VCCA, U1.VCCA_2, U1.VCCB, U1.VCCB_2
- new net 3P3AUX: C1.1, J1D.3P3VAUX@D32, U2.VCC
- new net 3P3V: C14.1, C2.1, C3.1, C4.1, C5.1, J1C.3P3V@C39, J1D.3P3V@D36, J1D.3P3V@D38, J1D.3P3V@D40, U1.2DIR, U1.VCCA, U1.VCCA_2, U5.EN, U5.IN
- new net CAM1_SCL: U3.SC1
- new net CAM1_SDA: U3.SD1
- new net CAM2_SCL: U3.SC0
- new net CAM2_SDA: U3.SD0
- new net EN#: U1.*1OE, U1.*2OE, U2.Y
- new net HDMI_SCL: U3.SC3
- new net HDMI_SDA: U3.SD3
- new net N$10: C12.1, U4.Y4
- new net N$11: C13.1, U4.Y5
- new net N$13: C15.1, U5.NR/FB
- new net N$2: LED1.A, R3.2
- new net N$3: U$8.1, U4.XIN/CLK
- new net N$5: U$8.2, U4.XOUT
- new net N$6: C8.1, R7.2, R8.2, U$10.2, U4.VDD
- new net N$7: R8.1, U4.S0
- new net N$8: R7.1, U4.VCTR
- new net N$9: C10.1, C11.1, U$12.2, U4.VDDOUT, U4.VDDOUT_2
- new net REG_1P8V: C16.1, U$10.1, U5.OUT
- new net TMDS_PLL_SCL: U3.SC2, U4.S2/SCL
- new net TMDS_PLL_SDA: U3.SD2, U4.S1/SDA
- new net VADJ: C6.1, C7.1, C9.1, J1G.VADJ@G39, J1H.VADJ@H40, R4.2, R5.2, R6.2, U$12.1, U1.VCCB, U1.VCCB_2, U3.VCC
- net FMC_CAM1_PCLK: now also U1.2B8
- net FMC_CAM1_PWDN: now also U1.1B2
- net FMC_CAM1_RST: now also U1.1B1
- net FMC_CAM1_RSVD5: now also U1.2B2
- net FMC_CAM2_PWDN: now also U1.1B8
- net FMC_CAM2_RST: now also U1.1B7
- net FMC_FRSTN_M2C_L: now also R1.2
- net GND: now also C1.2, C10.2, C11.2, C14.2, C15.2, C16.2, C2.2, C3.2, C4.2, C5.2, C6.2, C7.2, C8.2, LED1.C, R1.1, R2.1, U1.1DIR, U2.GND, U3.A0, U3.A1, U3.A2, U3.GND, U4.GND, U4.GND_2, U5.GND
- net I2C_SW_RST: now also R4.1, U3.*RESET
- net MUX_SCL: now also R6.1, U3.SCL
- net MUX_SDA: now also R5.1, U3.SDA
- net PG_C2M: now also R2.2, R3.1, U2.A

Commit message: update board schematic
Parts:
- removed C1: (no value), resistor:C-EUC0603
- removed C9: (no value), my-rcl:C-EUC0603
- removed R4, R5, R6: (no value), resistor:R-EU_R0603
- removed U$8: (no value), CX5032GB (CX-53F):CX5032GB27000
- added C101: 100nF, resistor:C-EUC0603
- added C200: 100nF, my-rcl:C-EUC0603
- added C305, C306, C307, C308, C309, C310, C311, C312, C313, C314, C315, C316, C503: 100nF, rcl:C-EUC0603
- added C500: 15nF, rcl:C-EUC0603
- added C501: 330pF, rcl:C-EUC0603
- added C502: 12pF, rcl:C-EUC0603
- added C507: 10uF 16V, rcl:C-EUC0603
- added C508: 47uF 10V, rcl:C-EUC0603
- added C509, C510: 2n2F, rcl:C-EUC0603
- added D1: MBRS130LT3, diode:MBRS130LT3
- added PAD1, PAD10, PAD11, PAD2, PAD3, PAD4, PAD5, PAD6, PAD7, PAD8, PAD9: (no value), wirepad:1,6/0,8
- added Q1: 27MHz, special:XTAL
- added R200, R201, R202, R203, R204, R205, R206, R207, R208, R209, R210: 4K7, resistor:R-EU_R0603
- added R500: 348K, rcl:R-EU_R0603
- added R501: 78K7, rcl:R-EU_R0603
- added R502: 40K2, rcl:R-EU_R0603
- added R503: 10K, rcl:R-EU_R0603
- added R504: 1K87, rcl:R-EU_R0603
- added R506: 36K5, rcl:R-EU_R0603
- added U$23, U$24: L-MY, my-rcl:L-MY
- added U6, U7: SN74AVCH16T245_DGV_48, SN74AVCH16T245_DGV_48:SN74AVCH16T245_DGV_48
- added U8: TPS54140_DGQ_10, TPS54140_DGQ_10:TPS54140_DGQ_10
- C102, C103, C104, C105, C106, C107, C201, C202, C203, C209, C210: value (none) -> 100nF
- C206, C208: value (none) -> 1uF
- C207: value (none) -> 10nF
- R105: value 4K7 -> 33R DNI
- R106: value 4K7 -> 4K7 DNI
- R211: value (none) -> 4K7 DNI
- R212: value (none) -> 4K7
- renumbered C10 to C202, C11 to C201, C12 to C209, C13 to C210, C14 to C206, C15 to C207, C16 to C208, C2 to C102, C3 to C103, C4 to C104, C5 to C105, C6 to C106, C7 to C107, C8 to C203, R1 to R104, R2 to R106, R3 to R105, R7 to R211, R8 to R212
Connections:
- new net CAM1_XCLK: C210.2
- new net CAM2_XCLK: C209.2
- new net N$15: C507.1, C510.1, R500.2, U$23.2, U8.VIN
- new net N$16: C503.1, U8.BOOT
- new net N$17: C503.2, D1.C, U$24.1, U8.PH
- new net N$19: R500.1, R501.2, U8.EN
- new net N$20: C500.1, U8.SS/TR
- new net N$21: R502.2, U8.RT/CLK
- new net N$22: J1H.FREF_A_M2C@H1, PAD1.P
- new net N$23: C502.1, R506.2, U8.COMP
- new net N$24: C501.1, R506.1
- new net N$25: R503.1, R504.2, U8.VSENSE
- new net N$26: J1D.GBTCLK0_M2C_P@D4, PAD3.P
- new net N$27: J1D.GBTCLK0_M2C_N@D5, PAD4.P
- new net N$28: J1D.TCK@D29, PAD5.P
- new net N$29: J1D.TMS@D33, PAD6.P
- new net N$30: J1D.TRST_L@D34, PAD7.P
- new net N$31: J1C.DP0_C2M_P@C2, PAD8.P
- new net N$32: J1C.DP0_C2M_N@C3, PAD9.P
- new net N$33: J1C.DP0_M2C_P@C6, PAD10.P
- new net N$34: J1C.DP0_M2C_N@C7, PAD11.P
- new net PGOOD: U8.PWRGD
- new net REG_5P0V: C508.1, R209.2, R210.2, R503.2, U$24.2
- net 12P0V: now also C509.1, U$23.1
- net 3P3AUX: now also C101.1; no longer C1.1
- net 3P3V: now also C305.1, C306.1, C309.1, C310.1, C313.1, C314.1, R202.2, R203.2, R205.2, R206.2, R207.2, R208.2, U6.1DIR, U6.2DIR, U6.VCCA, U6.VCCA_2, U7.1DIR, U7.2DIR, U7.VCCA, U7.VCCA_2
- net CAM1_SCL: now also R203.1
- net CAM1_SDA: now also R202.1
- net CAM2_SCL: now also R206.1
- net CAM2_SDA: now also R205.1
- net EN#: now also U6.*1OE, U6.*2OE, U7.*1OE, U7.*2OE
- net FMC_CAM1_D0: now also U6.2B4
- net FMC_CAM1_D1: now also U6.2B3
- net FMC_CAM1_D2: now also U6.2B2
- net FMC_CAM1_D3: now also U6.2B1
- net FMC_CAM1_D4: now also U6.1B8
- net FMC_CAM1_D5: now also U6.1B7
- net FMC_CAM1_D6: now also U6.1B6
- net FMC_CAM1_D7: now also U6.1B5
- net FMC_CAM1_D8: now also U6.1B4
- net FMC_CAM1_D9: now also U6.1B3
- net FMC_CAM1_HREF: now also U6.1B2
- net FMC_CAM1_VSYNC: now also U6.1B1
- net FMC_CAM2_D0: now also U7.2B8
- net FMC_CAM2_D1: now also U7.2B7
- net FMC_CAM2_D2: now also U7.2B6
- net FMC_CAM2_D3: now also U7.2B5
- net FMC_CAM2_D4: now also U7.2B4
- net FMC_CAM2_D5: now also U7.2B3
- net FMC_CAM2_D6: now also U7.2B2
- net FMC_CAM2_D7: now also U7.2B1
- net FMC_CAM2_D8: now also U7.1B8
- net FMC_CAM2_D9: now also U7.1B7
- net FMC_CAM2_HREF: now also U7.1B6
- net FMC_CAM2_PCLK: now also U7.1B4
- net FMC_CAM2_RSVD0: now also U7.1B3
- net FMC_CAM2_RSVD1: now also U7.1B2
- net FMC_CAM2_RSVD2: now also U7.1B1
- net FMC_CAM2_RSVD3: now also U6.2B8
- net FMC_CAM2_RSVD4: now also U6.2B7
- net FMC_CAM2_RSVD5: now also U6.2B6
- net FMC_CAM2_RSVD6: now also U6.2B5
- net FMC_CAM2_VSYNC: now also U7.1B5
- net GND: now also C101.2, C200.2, C305.2, C306.2, C307.2, C308.2, C309.2, C310.2, C311.2, C312.2, C313.2, C314.2, C315.2, C316.2, C500.2, C501.2, C502.2, C507.2, C508.2, C509.2, C510.2, D1.A, R501.1, R502.1, R504.1, U6.GND, U6.GND_2, U6.GND_3, U6.GND_4, U6.GND_5, U6.GND_6, U6.GND_7, U6.GND_8, U7.GND, U7.GND_2, U7.GND_3, U7.GND_4, U7.GND_5, U7.GND_6, U7.GND_7, U7.GND_8, U8.GND; no longer C1.2
- net HDMI_SCL: now also R210.1
- net HDMI_SDA: now also R209.1
- net I2C_SW_RST: now also R204.1; no longer R4.1
- net MUX_SCL: now also R200.1; no longer R6.1
- net MUX_SDA: now also R201.1; no longer R5.1
- net N$1: now also PAD2.P
- net N$3: now also Q1.1; no longer U$8.1
- net N$5: now also Q1.2; no longer U$8.2
- net TMDS_PLL_SCL: now also R208.1
- net TMDS_PLL_SDA: now also R207.1
- net VADJ: now also C200.1, C307.1, C308.1, C311.1, C312.1, C315.1, C316.1, R200.2, R201.2, R204.2, U6.VCCB, U6.VCCB_2, U7.VCCB, U7.VCCB_2; no longer C9.1, R4.2, R5.2, R6.2
